File: PCB/kicad/STM32_ExpUtilitia/STM32_ExpUtilitia.kicad_pcb (KiCad board)
At the start: 2 copper layers, 9 parts, among them J1 Conn_02x23_Odd_Even, J2 Conn_02x23_Odd_Even, SW1 KEY_UP, SW2 KEY0, SW3 KEY1

Commit message: update pcb schema and layout
Parts:
- J1, J2: value Conn_02x23_Odd_Even -> Conn_02x15_Odd_Even; footprint Connector_PinSocket_2.54mm:PinSocket_2x23_P2.54mm_Vertical -> Connector_PinHeader_2.54mm:PinHeader_2x15_P2.54mm_Vertical
- moved R1 126.1 mm to (147.3, 58.4), turned to 90 degrees
- moved R2 118.2 mm to (147.3, 68.6), turned to -90 degrees
- moved D1 107.7 mm to (152.4, 53.3)
- moved SW1 93.9 mm to (88.9, 62.9), turned to 180 degrees
- moved D2 56.8 mm to (152.4, 73.7)
- moved SW2 46.5 mm to (82.4, 73.7)
- moved SW3 43.0 mm to (82.4, 88.9)
- moved J1 32.3 mm to (96.5, 53.3)
- moved J2 10.9 mm to (139.7, 53.3)
Connections:
- D1 pad 1: /PB5 -> Net-(D1-K)
- D1 pad 2: Net-(D1-A) -> /5V
- D2 pad 1: /PE5 -> Net-(D2-K)
- D2 pad 2: Net-(D2-A) -> /5V
- J1 pad 1: /5V -> /3V3
- J1 pad 15: unconnected-(J1-Pin_15-Pad15) -> /PA5
- J1 pad 17: unconnected-(J1-Pin_17-Pad17) -> /PA3
- J1 pad 19: unconnected-(J1-Pin_19-Pad19) -> /PA1
- J1 pad 2: unconnected-(J1-Pin_2-Pad2) -> /3V3
- J1 pad 3: unconnected-(J1-Pin_3-Pad3) -> /3V3
- J1 pad 30: unconnected-(J1-Pin_30-Pad30) -> /GND
- J1 pad 4: unconnected-(J1-Pin_4-Pad4) -> /3V3
- J2 pad 1: unconnected-(J2-Pin_1-Pad1) -> /5V
- J2 pad 10: unconnected-(J2-Pin_10-Pad10) -> /PC8
- J2 pad 3: unconnected-(J2-Pin_3-Pad3) -> /GND
- J2 pad 4: unconnected-(J2-Pin_4-Pad4) -> /GND
- J2 pad 8: unconnected-(J2-Pin_8-Pad8) -> /PC6
- R1 pad 1: Net-(D1-A) -> /PC6
- R1 pad 2: +3V3 -> Net-(D1-K)
- R2 pad 1: Net-(D2-A) -> /PC8
- R2 pad 2: +3V3 -> Net-(D2-K)
- SW1 pad 1: /PA0 -> /PA5
- SW1 pad 2: +3V3 -> /3V3
- SW2 pad 1: /PE4 -> /PA3
- SW2 pad 2: GND -> /GND
- SW3 pad 1: /PE3 -> /PA1
- SW3 pad 2: GND -> /GND
Routing:
- net /GND: track 0.00 -> 47.1 mm
- net /5V: track 0.00 -> 38.7 mm
- net /PA1: track 0.00 -> 17.3 mm
- net /PA5: track 0.00 -> 12.5 mm
- net /3V3: track 0.00 -> 10.2 mm
- net /PC8: track 0.00 -> 8.67 mm
- net /PA3: track 0.00 -> 7.62 mm
- net /PC6: track 0.00 -> 6.13 mm
- net Net-(D2-K): track 0.00 -> 5.08 mm
- net Net-(D1-K): track 0.00 -> 5.08 mm
Other:
- board outline added: 83.8 x 71.1 mm
