File: PCB/kicad/STM32_ExpUtilitia/STM32_ExpUtilitia.kicad_sch (KiCad schematic)
At the start: 9 parts, among them J1 Conn_02x23_Odd_Even, J2 Conn_02x23_Odd_Even, SW1 KEY_UP, SW2 KEY0, SW3 KEY1

Commit message: update pcb schema and layout
Parts:
- removed J1, J2: Conn_02x23_Odd_Even, Connector_PinSocket_2.54mm:PinSocket_2x23_P2.54mm_Vertical, symbol Connector_Generic:Conn_02x23_Odd_Even
- added J1, J2: Conn_02x15_Odd_Even, Connector_PinHeader_2.54mm:PinHeader_2x15_P2.54mm_Vertical, symbol Connector_Generic:Conn_02x15_Odd_Even
Connections:
- net 5V: now also D1.2 (A), D2.2 (A), J2.1 (Pin_1), J2.2 (Pin_2)
- net GND: now also J1.30 (Pin_30), J2.3 (Pin_3), J2.4 (Pin_4)
- net PC6: now reaches R1.1
- net PC6: now also J2.8 (Pin_8); no longer D1.2 (A)
- net PC8: now reaches R2.1
- net PC8: now also J2.10 (Pin_10); no longer D2.2 (A)
- removed net +3V3: R1.2, R2.2, SW1.2
- net PA0 renamed PA5
- net PA5: now also J1.15 (Pin_15)
- net PB5: no longer names the net of D1.1 (K)
- net PB5: now also R1.2
- net PE3 renamed PA1
- net PA1: now also J1.19 (Pin_19)
- net PE4 renamed PA3
- net PA3: now also J1.17 (Pin_17)
- net PE5: no longer names the net of D2.1 (K)
- net PE5: now also R2.2
- new net 3V3: J1.1 (Pin_1), J1.2 (Pin_2), J1.3 (Pin_3), J1.4 (Pin_4), SW1.2
- no-connect marks 85 -> 46
